File: KiCad/65C816_SBC.kicad_sch (KiCad schematic)
At the start: 50 parts, among them J0 JTAG, J1 EXPANSION, J2 PA, SW0 RESET, SW1 NMI, U1 FT240XS, U10 DS1813-10, U11 DS1813-10, U3 ATF1508AS, U4 W65C22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

Commit message: Updating the Project
Most things stayed the same, but mainly the BIOS now has a splash screen when first powering it up.
Parts:
- BJ0: value (none) -> POWER; footprint (none) -> Connector_BarrelJack:BarrelJack_Horizontal
- C1: value (none) -> 47pF
- C3: value (none) -> 0.1uF
- C4: value (none) -> 100uF
- J3: value (none) -> PB; footprint (none) -> Connector_PinHeader_2.54mm:PinHeader_1x03_P2.54mm_Vertical
- R0, R1: value (none) -> 27
- R3: value (none) -> 3.3k; footprint (none) -> Resistor_THT:R_Axial_DIN0207_L6.3mm_D2.5mm_P2.54mm_Vertical
- R4: footprint (none) -> Resistor_THT:R_Axial_DIN0207_L6.3mm_D2.5mm_P2.54mm_Vertical
- RN0: value (none) -> 3.3k
- U0: value (none) -> LM340T; footprint (none) -> Package_TO_SOT_THT:TO-220-3_Vertical
- U2: value (none) -> 74AC74; footprint (none) -> Package_DIP:DIP-14_W7.62mm_Socket
- U5: footprint (none) -> Package_LCC:PLCC-32_THT-Socket
- U9: value (none) -> 74ACT245; footprint (none) -> Package_DIP:DIP-20_W7.62mm_Socket
- X0: value (none) -> 50MHz; footprint (none) -> Oscillator:Oscillator_DIP-8
Connections:
- net 3V3: now also U1.16 (~{RESET})
- no-connect marks 11 -> 10
Changed lines of the file:
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@@
   (no_connect (at 151.13 195.58))
   (no_connect (at 50.8 71.12))
-  (no_connect (at 158.75 44.45))
   (no_connect (at 104.14 99.06))
   (no_connect (at 251.46 35.56))
@@
     (stroke (width 0) (type default) (color 0 0 0 0))
   )
+  (wire (pts (xy 156.21 44.45) (xy 158.75 44.45))
+    (stroke (width 0) (type default) (color 0 0 0 0))
+  )
   (bus (pts (xy 285.75 196.85) (xy 285.75 199.39))
     (stroke (width 0) (type default) (color 0 0 0 0))
@@
     (stroke (width 0) (type default) (color 0 0 0 0))
   )
+  (wire (pts (xy 151.13 29.21) (xy 158.75 29.21))
+    (stroke (width 0) (type default) (color 0 0 0 0))
+  )
   (wire (pts (xy 30.48 245.11) (xy 33.02 245.11))
     (stroke (width 0) (type default) (color 0 0 0 0))
@@
     (stroke (width 0) (type default) (color 0 0 0 0))
   )
-  (wire (pts (xy 151.13 29.21) (xy 158.75 29.21))
-    (stroke (width 0) (type default) (color 0 0 0 0))
-  )
   (wire (pts (xy 346.71 207.01) (xy 356.87 207.01))
     (stroke (width 0) (type default) (color 0 0 0 0))
@@
     (effects (font (size 1.27 1.27)) (justify left bottom))
   )
+  (label "3V3" (at 156.21 44.45 180)
+    (effects (font (size 1.27 1.27)) (justify right bottom))
+  )
   (label "A7" (at 354.33 217.17 180)
     (effects (font (size 1.27 1.27)) (justify right bottom))
@@
       (effects (font (size 1.27 1.27)) (justify left))
     )
-    (property "Value" "" (id 1) (at 136.6394 63.6071 0)
+    (property "Value" "74AC74" (id 1) (at 136.6394 63.6071 0)
       (effects (font (size 1.27 1.27)) (justify left))
     )
-    (property "Footprint" "" (id 2) (at 134.62 69.85 0)
+    (property "Footprint" "Package_DIP:DIP-14_W7.62mm_Socket" (id 2) (at 134.62 69.85 0)
       (effects (font (size 1.27 1.27)) hide)
     )
@@
       (effects (font (size 1.27 1.27)) (justify left))
     )
-    (property "Value" "" (id 1) (at 126.492 141.4022 0)
+    (property "Value" "PB" (id 1) (at 126.492 141.4022 0)
       (effects (font (size 1.27 1.27)) (justify left))
     )
-    (property "Footprint" "" (id 2) (at 124.46 139.7 0)
+    (property "Footprint" "Connector_PinHeader_2.54mm:PinHeader_1x03_P2.54mm_Vertical" (id 2) (at 124.46 139.7 0)
       (effects (font (size 1.27 1.27)) hide)
     )
@@
     (property "Reference" "R4" (id 0) (at 26.67 242.57 90))
     (property "Value" "3.3k" (id 1) (at 26.67 245.11 90))
-    (property "Footprint" "" (id 2) (at 26.67 246.888 90)
+    (property "Footprint" "Resistor_THT:R_Axial_DIN0207_L6.3mm_D2.5mm_P2.54mm_Vertical" (id 2) (at 26.67 246.888 90)
       (effects (font (size 1.27 1.27)) hide)
     )
@@
       (effects (font (size 1.27 1.27)) (justify right))
     )
-    (property "Value" "" (id 1) (at 197.3706 200.7671 0)
+    (property "Value" "74ACT245" (id 1) (at 197.3706 200.7671 0)
       (effects (font (size 1.27 1.27)) (justify right))
     )
-    (property "Footprint" "" (id 2) (at 196.85 217.17 0)
+    (property "Footprint" "Package_DIP:DIP-20_W7.62mm_Socket" (id 2) (at 196.85 217.17 0)
       (effects (font (size 1.27 1.27)) hide)
     )
@@
       (effects (font (size 1.27 1.27)) (justify left))
     )
-    (property "Value" "" (id 1) (at 36.83 31.75 0)
+    (property "Value" "0.1uF" (id 1) (at 36.83 31.75 0)
       (effects (font (size 1.27 1.27)) (justify right))
     )
@@
       (effects (font (size 1.27 1.27)) (justify left))
     )
-    (property "Value" "" (id 1) (at 111.76 33.02 0)
+    (property "Value" "47pF" (id 1) (at 111.76 33.02 0)
       (effects (font (size 1.27 1.27)) (justify left))
     )
@@
     (in_bom yes) (on_board yes) (fields_autoplaced)
     (property "Reference" "U0" (id 0) (at 46.99 32.4952 0))
-    (property "Value" "" (id 1) (at 46.99 35.0321 0))
-    (property "Footprint" "" (id 2) (at 46.99 32.385 0)
+    (property "Value" "LM340T" (id 1) (at 46.99 35.0321 0))
+    (property "Footprint" "Package_TO_SOT_THT:TO-220-3_Vertical" (id 2) (at 46.99 32.385 0)
       (effects (font (size 1.27 1.27) italic) hide)
     )
@@
     (in_bom yes) (on_board yes)
     (property "Reference" "R0" (id 0) (at 140.97 34.29 90))
-    (property "Value" "" (id 1) (at 140.97 36.83 90))
+    (property "Value" "27" (id 1) (at 140.97 36.83 90))
     (property "Footprint" "Resistor_THT:R_Axial_DIN0207_L6.3mm_D2.5mm_P2.54mm_Vertical" (id 2) (at 140.97 38.608 90)
       (effects (font (size 1.27 1.27)) hide)
@@
       (effects (font (size 1.27 1.27)) (justify left))
     )
-    (property "Value" "" (id 1) (at 136.6394 92.8171 0)
+    (property "Value" "74AC74" (id 1) (at 136.6394 92.8171 0)
       (effects (font (size 1.27 1.27)) (justify left))
     )
-    (property "Footprint" "" (id 2) (at 134.62 99.06 0)
+    (property "Footprint" "Package_DIP:DIP-14_W7.62mm_Socket" (id 2) (at 134.62 99.06 0)
       (effects (font (size 1.27 1.27)) hide)
     )
@@
       (effects (font (size 1.27 1.27)) (justify left))
     )
-    (property "Value" "" (id 1) (at 59.69 31.75 0)
+    (property "Value" "100uF" (id 1) (at 59.69 31.75 0)
       (effects (font (size 1.27 1.27)) (justify right))
     )
@@
     (in_bom yes) (on_board yes)
     (property "Reference" "X0" (id 0) (at 116.84 90.17 0))
-    (property "Value" "" (id 1) (at 116.84 92.71 0))
-    (property "Footprint" "" (id 2) (at 123.19 107.95 0)
+    (property "Value" "50MHz" (id 1) (at 116.84 92.71 0))
+    (property "Footprint" "Oscillator:Oscillator_DIP-8" (id 2) (at 123.19 107.95 0)
       (effects (font (size 1.27 1.27)) hide)
     )
@@
       (effects (font (size 1.27 1.27)) (justify left))
     )
-    (property "Value" "" (id 1) (at 49.022 136.5762 0)
+    (property "Value" "3.3k" (id 1) (at 49.022 136.5762 0)
       (effects (font (size 1.27 1.27)) (justify left))
     )
@@
     (property "Reference" "U5" (id 0) (at 252.73 173.99 0))
     (property "Value" "SST39SF040" (id 1) (at 252.73 176.53 0))
-    (property "Footprint" "" (id 2) (at 252.73 175.26 0)
+    (property "Footprint" "Package_LCC:PLCC-32_THT-Socket" (id 2) (at 252.73 175.26 0)
       (effects (font (size 1.27 1.27)) hide)
     )
@@
     (in_bom yes) (on_board yes)
     (property "Reference" "R1" (id 0) (at 140.97 41.91 90))
-    (property "Value" "" (id 1) (at 140.97 39.37 90))
+    (property "Value" "27" (id 1) (at 140.97 39.37 90))
     (property "Footprint" "Resistor_THT:R_Axial_DIN0207_L6.3mm_D2.5mm_P2.54mm_Vertical" (id 2) (at 140.97 41.148 90)
       (effects (font (size 1.27 1.27)) hide)
@@
     (in_bom yes) (on_board yes)
     (property "Reference" "R3" (id 0) (at 26.67 223.52 90))
-    (property "Value" "" (id 1) (at 26.67 226.06 90))
-    (property "Footprint" "" (id 2) (at 26.67 227.838 90)
+    (property "Value" "3.3k" (id 1) (at 26.67 226.06 90))
+    (property "Footprint" "Resistor_THT:R_Axial_DIN0207_L6.3mm_D2.5mm_P2.54mm_Vertical" (id 2) (at 26.67 227.838 90)
       (effects (font (size 1.27 1.27)) hide)
     )
@@
       (effects (font (size 1.27 1.27)) (justify left))
     )
-    (property "Value" "" (id 1) (at 79.502 184.5822 0)
+    (property "Value" "74AC74" (id 1) (at 79.502 184.5822 0)
       (effects (font (size 1.27 1.27)) (justify left))
     )
-    (property "Footprint" "" (id 2) (at 73.66 182.88 0)
+    (property "Footprint" "Package_DIP:DIP-14_W7.62mm_Socket" (id 2) (at 73.66 182.88 0)
       (effects (font (size 1.27 1.27)) hide)
     )
@@
     (in_bom yes) (on_board yes) (fields_autoplaced)
     (property "Reference" "BJ0" (id 0) (at 24.13 33.1302 0))
-    (property "Value" "" (id 1) (at 24.13 35.6671 0))
-    (property "Footprint" "" (id 2) (at 25.4 41.656 0)
+    (property "Value" "POWER" (id 1) (at 24.13 35.6671 0))
+    (property "Footprint" "Connector_BarrelJack:BarrelJack_Horizontal" (id 2) (at 25.4 41.656 0)
       (effects (font (size 1.27 1.27)) hide)
     )
